Commit message: dynamic collision avoidance almost working

File: gym_pybullet_drones/assets/red_cylinder.urdf (robot description, URDF)
Before this commit: robot red_cylinder, 1 links, 0 joints
Links:
- link cylinder_link: geometry collision cylinder length=5.0 radius=0.3; visual cylinder length=5.0 radius=0.3
