Commit message: dynamic planning working: 29/50 successful runs with 20 obstacles

File: gym_pybullet_drones/assets/mantis.urdf (robot description, URDF)
Before this commit: robot cf2, 6 links, 5 joints
Links:
- link base_link: geometry collision cylinder length=.1 radius=.3; visual mesh filename=./yunque.dae scale=1 1 1
